Commit message: made original file copies

File: rb1_ros2_description/xacro/rb1_ros2_base.urdf_backup.xacro (robot description, xacro)
@@ -1,5 +1,5 @@
 <?xml version="1.0"?>
-<robot name="rb1_base" xmlns:xacro="http://www.ros.org/wiki/xacro">
-<xacro:property name="robot_name" value="$(arg robot_name)"/>
+<robot name="rb1_base"
+	xmlns:xacro="http://www.ros.org/wiki/xacro">
 	<!-- ***************** -->
 	<!-- Imported elements -->
@@ -84,48 +84,5 @@
 		<origin xyz="0.234 0.0 0.092" rpy="0 0 0"/>
 	</xacro:sensor_orbbec_astra>
-    <!-- <gazebo>
-        <plugin name="box_bot_joint_state" filename="libgazebo_ros_joint_state_publisher.so">
-        <ros>
-            <namespace>/${robot_name}</namespace>
-            <remapping>~/out:=joint_states</remapping>
-        </ros>
-        <update_rate>30</update_rate>
-        <joint_name>robot_left_wheel_joint</joint_name>
-        <joint_name>robot_right_wheel_joint</joint_name>
-        <joint_name>robot_elevator_platform_joint</joint_name>
-        </plugin>
-    </gazebo> -->
 	<!-- Gazebo ros2 control plugins -->
-    <!-- <ros2_control name='GazeboSystem' type='system'>
-      <hardware>
-        <plugin>gazebo_ros2_control/GazeboSystem</plugin>
-      </hardware>
-      <ros>
-        <namespace>/${robot_name}</namespace>
-        <remapping>/cmd_vel:=cmd_vel_unstamped</remapping>
-      </ros>
-      <joint name='robot_left_wheel_joint'>
-        <command_interface name='velocity'>
-          <param name='min'>-10</param>
-          <param name='max'>10</param>
-        </command_interface>
-        <state_interface name='velocity'/>
-        <state_interface name='position'/>
-      </joint>
-      <joint name='robot_right_wheel_joint'>
-        <command_interface name='velocity'>
-          <param name='min'>-10</param>
-          <param name='max'>10</param>
-        </command_interface>
-        <state_interface name='velocity'/>
-        <state_interface name='position'/>
-      </joint>
-    </ros2_control> -->
 	<!-- <xacro:ros2_control/> -->
-  <!-- <gazebo>
-    <plugin name='gazebo_ros2_control' filename='libgazebo_ros2_control.so'>
-      <robot_sim_type>gazebo_ros2_control/GazeboSystem</robot_sim_type>
-      <parameters>$(find rb1_ros2_description)/config/rb1_controller.yaml</parameters>
-    </plugin>
-  </gazebo> -->
 </robot>
