Commit message: add joint state publisher to xacro file and it works

File: rb1_ros2_description/xacro/rb1_ros2_base.urdf.xacro (robot description, xacro)
@@ -1,5 +1,5 @@
 <?xml version="1.0"?>
-<robot name="rb1_base"
-	xmlns:xacro="http://www.ros.org/wiki/xacro">
+<robot name="rb1_base" xmlns:xacro="http://www.ros.org/wiki/xacro">
+<xacro:property name="robot_name" value="$(arg robot_name)"/>
 	<!-- ***************** -->
 	<!-- Imported elements -->
@@ -84,5 +84,47 @@
 		<origin xyz="0.234 0.0 0.092" rpy="0 0 0"/>
 	</xacro:sensor_orbbec_astra>
+    <gazebo>
+        <plugin name="box_bot_joint_state" filename="libgazebo_ros_joint_state_publisher.so">
+        <ros>
+            <namespace>/${robot_name}</namespace>
+            <remapping>~/out:=joint_states</remapping>
+        </ros>
+        <update_rate>30</update_rate>
+        <joint_name>robot_left_wheel_joint</joint_name>
+        <joint_name>robot_right_wheel_joint</joint_name>
+        </plugin>
+    </gazebo>
 	<!-- Gazebo ros2 control plugins -->
+    <ros2_control name='GazeboSystem' type='system'>
+      <hardware>
+        <plugin>gazebo_ros2_control/GazeboSystem</plugin>
+      </hardware>
+      <ros>
+        <namespace>/${robot_name}</namespace>
+        <remapping>/cmd_vel:=cmd_vel</remapping>
+      </ros>
+      <joint name='robot_left_wheel_joint'>
+        <command_interface name='velocity'>
+          <param name='min'>-10</param>
+          <param name='max'>10</param>
+        </command_interface>
+        <state_interface name='velocity'/>
+        <state_interface name='position'/>
+      </joint>
+      <joint name='robot_right_wheel_joint'>
+        <command_interface name='velocity'>
+          <param name='min'>-10</param>
+          <param name='max'>10</param>
+        </command_interface>
+        <state_interface name='velocity'/>
+        <state_interface name='position'/>
+      </joint>
+    </ros2_control>
 	<!-- <xacro:ros2_control/> -->
+  <gazebo>
+    <plugin name='gazebo_ros2_control' filename='libgazebo_ros2_control.so'>
+      <robot_sim_type>gazebo_ros2_control/GazeboSystem</robot_sim_type>
+      <parameters>$(find rb1_ros2_description)/config/rb1_controller.yaml</parameters>
+    </plugin>
+  </gazebo>
 </robot>

Commit message: added position controller but I am aware of how to handle name space

File: rb1_ros2_description/xacro/rb1_ros2_base.urdf.xacro (robot description, xacro)
@@ -97,5 +97,5 @@
     </gazebo> -->
 	<!-- Gazebo ros2 control plugins -->
-    <!-- <ros2_control name='GazeboSystem' type='system'>
+    <ros2_control name='GazeboSystem' type='system'>
       <hardware>
         <plugin>gazebo_ros2_control/GazeboSystem</plugin>
@@ -121,11 +121,32 @@
         <state_interface name='position'/>
       </joint>
-    </ros2_control> -->
+    </ros2_control>
 	<!-- <xacro:ros2_control/> -->
-  <!-- <gazebo>
+  <gazebo>
     <plugin name='gazebo_ros2_control' filename='libgazebo_ros2_control.so'>
       <robot_sim_type>gazebo_ros2_control/GazeboSystem</robot_sim_type>
       <parameters>$(find rb1_ros2_description)/config/rb1_controller.yaml</parameters>
     </plugin>
-  </gazebo> -->
+  </gazebo>
+  <!-- Adding position control -->
+  <!-- <xacro:ros2_control/> -->
+  <ros2_control name="position_controllers_exercise" type="system">
+    <hardware>
+      <plugin>gazebo_ros2_control/GazeboSystem</plugin>
+    </hardware>
+    <joint name="lift_joint">
+      <command_interface name="position">
+        <param name="min">-2.0</param>
+        <param name="max">0</param>
+      </command_interface>
+      <state_interface name="position"/>
+      <state_interface name="velocity"/>
+      <state_interface name="effort"/>
+    </joint>
+  </ros2_control>
+  <gazebo>
+    <plugin filename="libgazebo_ros2_control.so" name="gazebo_ros2_control">
+      <parameters>$(find rb1_ros2_description)/config/position_controller_config.yaml</parameters>
+    </plugin>
+  </gazebo>
 </robot>

Commit message: learning from previous session

File: rb1_ros2_description/xacro/rb1_ros2_base.urdf.xacro (robot description, xacro)
@@ -84,6 +84,6 @@
 		<origin xyz="0.234 0.0 0.092" rpy="0 0 0"/>
 	</xacro:sensor_orbbec_astra>
-    <!-- <gazebo>
-        <plugin name="box_bot_joint_state" filename="libgazebo_ros_joint_state_publisher.so">
+    <gazebo>
+        <plugin name="rb1_joint_state" filename="libgazebo_ros_joint_state_publisher.so">
         <ros>
             <namespace>/${robot_name}</namespace>
@@ -95,5 +95,5 @@
         <joint_name>robot_elevator_platform_joint</joint_name>
         </plugin>
-    </gazebo> -->
+    </gazebo>
 	<!-- Gazebo ros2 control plugins -->
     <ros2_control name='GazeboSystem' type='system'>
@@ -129,23 +129,35 @@
     </plugin>
   </gazebo>
-  <!-- Adding position control -->
-  <!-- <xacro:ros2_control/> -->
-  <ros2_control name="position_controllers_exercise" type="system">
-    <hardware>
-      <plugin>gazebo_ros2_control/GazeboSystem</plugin>
-    </hardware>
-    <joint name="lift_joint">
-      <command_interface name="position">
-        <param name="min">-2.0</param>
-        <param name="max">0</param>
-      </command_interface>
-      <state_interface name="position"/>
-      <state_interface name="velocity"/>
-      <state_interface name="effort"/>
-    </joint>
-  </ros2_control>
+	<!-- Gazebo ros2 control plugins -->
+    <ros2_control name='GazeboSystem' type='system'>
+      <hardware>
+        <plugin>gazebo_ros2_control/GazeboSystem</plugin>
+      </hardware>
+      <ros>
+        <namespace>/${robot_name}</namespace>
+        <remapping>/cmd_vel:=cmd_vel</remapping>
+      </ros>
+      <joint name='robot_left_wheel_joint'>
+        <command_interface name='velocity'>
+          <param name='min'>-10</param>
+          <param name='max'>10</param>
+        </command_interface>
+        <state_interface name='velocity'/>
+        <state_interface name='position'/>
+      </joint>
+      <joint name='robot_right_wheel_joint'>
+        <command_interface name='velocity'>
+          <param name='min'>-10</param>
+          <param name='max'>10</param>
+        </command_interface>
+        <state_interface name='velocity'/>
+        <state_interface name='position'/>
+      </joint>
+    </ros2_control>
+	<!-- <xacro:ros2_control/> -->
   <gazebo>
-    <plugin filename="libgazebo_ros2_control.so" name="gazebo_ros2_control">
-      <parameters>$(find rb1_ros2_description)/config/position_controller_config.yaml</parameters>
+    <plugin name='gazebo_ros2_control' filename='libgazebo_ros2_control.so'>
+      <robot_sim_type>gazebo_ros2_control/GazeboSystem</robot_sim_type>
+      <parameters>$(find rb1_ros2_description)/config/rb1_controller.yaml</parameters>
     </plugin>
   </gazebo>
