Commit message: removing robot name space and it works.. but it is remained at unclaimed

File: rb1_ros2_description/xacro/rb1_ros2_base.urdf copy.xacro (robot description, xacro)
@@ -1,4 +1,6 @@
 <?xml version="1.0"?>
 <robot name="rb1_robot" xmlns:xacro="http://www.ros.org/wiki/xacro">
+<xacro:property name="robot_name" value="$(arg robot_name)"/>
+<!-- <xacro:arg name="robot_name" default="rb1_robot"/> -->
 	<!-- ***************** -->
 	<!-- Imported elements -->
@@ -100,4 +102,8 @@
         <plugin>gazebo_ros2_control/GazeboSystem</plugin>
       </hardware>
+      <ros>
+        <namespace>/${robot_name}</namespace>
+        <remapping>/cmd_vel:=cmd_vel_unstamped</remapping>
+      </ros>
       <joint name='robot_left_wheel_joint'>
         <command_interface name='velocity'>
@@ -131,7 +137,8 @@
     <gazebo>
         <plugin name="gazebo_ros2_control" filename="libgazebo_ros2_control.so">
+            <namespace>/${robot_name}</namespace>
             <robot_sim_type>gazebo_ros2_control/GazeboSystem</robot_sim_type>
             <robot_param>robot_description</robot_param>
-            <robot_param_node>/robot_state_publisher</robot_param_node>
+            <robot_param_node>/rb1_robot/robot_state_publisher</robot_param_node>
             <parameters>$(find rb1_ros2_description)/config/rb1_controller.yaml</parameters>
             <!-- <robotSimType>gazebo_ros2_control/DefaultRobotHWSim</robotSimType> -->
