Commit message: add all files and commit

File: rb1_ros2_description/urdf/elevator/elevator.urdf.xacro (robot description, xacro)
@@ -61,5 +61,6 @@
 			<axis xyz="0 0 1"/>
 			<limit effort="10.0" lower="0.0" upper="0.034" velocity="0.5"/>
-	</joint>
+            <dynamics damping="0.1" friction="1.0"/>
+    </joint>
 	<link name="${prefix}_platform_link">
 		<!--inertial>
